File: ISA8019.sch (KiCad schematic (older format))
At the start: 56 parts, among them J1 Bus_ISA_16bit, J2 8P8C_Shielded, J4 Jumper mode, J5 PNP force, J6 BROM size and base address, J7 I/O base address, J8 Medium type, J9 IRQ select, T1 13F-39MNL, U1 RTL8019AS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

Commit message: 8 bit network card variant
Parts:
- removed H2: MountingHole, ToolingHole:ToolingHole_JLCSMT, symbol Mechanical:MountingHole
- removed J1: Bus_ISA_16bit, Bus_AT_without_Silkscreen:BUS_AT_WO_SILKSCREEN, symbol Connector:Bus_ISA_16bit
- added J1: Bus_ISA_8bit, My_Components:Conn_Edge_PCB_ISA8, symbol Connector:Bus_ISA_8bit
Connections:
- net +12V: now also J1.9 (+12V)
- net +5V: now also J1.29 (VCC), J1.3 (VCC)
- net GND: now also J1.1 (GND), J1.10 (GND), J1.31 (GND)
- net ISA_A0: now also J1.62 (BA00)
- net ISA_A1: now also J1.61 (BA01)
- net ISA_A10: now also J1.52 (BA10)
- net ISA_A11: now also J1.51 (BA11)
- net ISA_A12: now also J1.50 (BA12)
- net ISA_A13: now also J1.49 (BA13)
- net ISA_A14: now also J1.48 (BA14)
- net ISA_A15: now also J1.47 (BA15)
- net ISA_A16: now also J1.46 (BA16)
- net ISA_A17: now also J1.45 (BA17)
- net ISA_A18: now also J1.44 (BA18)
- net ISA_A19: now also J1.43 (BA19)
- net ISA_A2: now also J1.60 (BA02)
- net ISA_A3: now also J1.59 (BA03)
- net ISA_A4: now also J1.58 (BA04)
- net ISA_A5: now also J1.57 (BA05)
- net ISA_A6: now also J1.56 (BA06)
- net ISA_A7: now also J1.55 (BA07)
- net ISA_A8: now also J1.54 (BA08)
- net ISA_A9: now also J1.53 (BA09)
- net ISA_AEN: now also J1.42 (AEN)
- net ISA_D0: now also J1.40 (DB0)
- net ISA_D1: now also J1.39 (DB1)
- net ISA_D2: now also J1.38 (DB2)
- net ISA_D3: now also J1.37 (DB3)
- net ISA_D4: now also J1.36 (DB4)
- net ISA_D5: now also J1.35 (DB5)
- net ISA_D6: now also J1.34 (DB6)
- net ISA_D7: now also J1.33 (DB7)
- net ISA_IO_CH_RDY: now also J1.41 (IO_READY)
- net ISA_IRQ2: now also J1.4 (IRQ2)
- net ISA_IRQ3: now also J1.25 (IRQ3)
- net ISA_IRQ4: now also J1.24 (IRQ4)
- net ISA_IRQ5: now also J1.23 (IRQ5)
- net ISA_IRQ6: now also J1.22 (IRQ6)
- net ISA_IRQ7: now also J1.21 (IRQ7)
- net ISA_RESET: now also J1.2 (RESET)
- net ~ISA_IOR: now also J1.14 (~IOR)
- net ~ISA_IOW: now also J1.13 (~IOW)
- net ~ISA_SMEMR: now also J1.12 (~SMEMR)
- net ~ISA_SMEMW: now also J1.11 (~SMEMW)
Other:
- moved on the sheet: C2
Changed lines of the file:
@@
 $EndDescr
-$Comp
-L Connector:Bus_ISA_16bit J1
-U 1 1 5FAD818A
-P 3000 4000
-F 0 "J1" H 3000 6767 50  0000 C CNN
-F 1 "Bus_ISA_16bit" H 3000 6676 50  0000 C CNN
-F 2 "Bus_AT_without_Silkscreen:BUS_AT_WO_SILKSCREEN" H 3000 4050 50  0001 C CNN
-F 3 "https://en.wikipedia.org/wiki/Industry_Standard_Architecture" H 3000 4050 50  0001 C CNN
-	1    3000 4000
-	1    0    0    -1
-$EndComp
 $Comp
 L RTL8019:RTL8019AS U1
@@
 Text Label 4050 2300 2    50   ~ 0
 ISA_D0
-Text Label 4050 5700 2    50   ~ 0
-ISA_D8
-Text Label 4050 5800 2    50   ~ 0
-ISA_D9
-Text Label 4050 5900 2    50   ~ 0
-ISA_D10
-Text Label 4050 6000 2    50   ~ 0
-ISA_D11
-Text Label 4050 6100 2    50   ~ 0
-ISA_D12
-Text Label 4050 6200 2    50   ~ 0
-ISA_D13
-Text Label 4050 6300 2    50   ~ 0
-ISA_D14
-Text Label 4050 6400 2    50   ~ 0
-ISA_D15
-Wire Wire Line
-	3700 5700 4050 5700
-Wire Wire Line
-	4050 5800 3700 5800
-Wire Wire Line
-	3700 5900 4050 5900
-Wire Wire Line
-	4050 6000 3700 6000
-Wire Wire Line
-	3700 6100 4050 6100
-Wire Wire Line
-	4050 6200 3700 6200
-Wire Wire Line
-	3700 6300 4050 6300
-Wire Wire Line
-	4050 6400 3700 6400
 Wire Wire Line
 	3700 1600 4050 1600
@@
 Wire Wire Line
 	1550 2400 2300 2400
-$Comp
-L power:GND #PWR0105
-U 1 1 5FB73D29
-P 1550 6600
-F 0 "#PWR0105" H 1550 6350 50  0001 C CNN
-F 1 "GND" H 1555 6427 50  0000 C CNN
-F 2 "" H 1550 6600 50  0001 C CNN
-F 3 "" H 1550 6600 50  0001 C CNN
-	1    1550 6600
-	1    0    0    -1
-$EndComp
 Wire Wire Line
 	1550 4500 2300 4500
@@
 Connection ~ 1550 2400
 Wire Wire Line
-	1550 6600 1550 6400
-Wire Wire Line
-	1550 6400 2300 6400
-Wire Wire Line
-	1550 6400 1550 4500
-Connection ~ 1550 6400
-Wire Wire Line
 	2300 4300 2000 4300
 Wire Wire Line
 	1750 1700 2300 1700
-$Comp
-L power:+5V #PWR0107
-U 1 1 5FBC7376
-P 2000 6200
-F 0 "#PWR0107" H 2000 6050 50  0001 C CNN
-F 1 "+5V" H 2015 6373 50  0000 C CNN
-F 2 "" H 2000 6200 50  0001 C CNN
-F 3 "" H 2000 6200 50  0001 C CNN
-	1    2000 6200
-	1    0    0    -1
-$EndComp
-Wire Wire Line
-	2300 6200 2000 6200
 $Comp
 L Ethernet_Transformer:13F-39MNL T?
@@
 $Comp
 L Mechanical:MountingHole H?
-U 1 1 5FC1F47E
-P 15250 9650
-AR Path="/5FBCDFD3/5FC1F47E" Ref="H?"  Part="1"
-AR Path="/5FC1F47E" Ref="H2"  Part="1"
-F 0 "H2" H 15350 9696 50  0000 L CNN
-F 1 "MountingHole" H 15350 9605 50  0000 L CNN
-F 2 "ToolingHole:ToolingHole_JLCSMT" H 15250 9650 50  0001 C CNN
-F 3 "~" H 15250 9650 50  0001 C CNN
-	1    15250 9650
-	1    0    0    -1
-$EndComp
-$Comp
-L Mechanical:MountingHole H?
 U 1 1 5FC1F484
 P 15250 9450
@@
 Wire Wire Line
 	1850 3900 2300 3900
-Text Label 1850 4900 0    50   ~ 0
-ISA_IRQ10
-Text Label 1850 5000 0    50   ~ 0
-ISA_IRQ11
-Text Label 1850 5100 0    50   ~ 0
-ISA_IRQ12
-Text Label 1850 5200 0    50   ~ 0
-ISA_IRQ15
-Text Label 1850 5300 0    50   ~ 0
-ISA_IRQ14
-Wire Wire Line
-	1850 4900 2300 4900
-Wire Wire Line
-	2300 5000 1850 5000
-Wire Wire Line
-	1850 5100 2300 5100
-Wire Wire Line
-	2300 5200 1850 5200
-Wire Wire Line
-	1850 5300 2300 5300
 Text Label 5150 3250 2    50   ~ 0
 ~ISA_IOCS16
-Text Label 1850 4800 0    50   ~ 0
-~ISA_IOCS16
-Wire Wire Line
-	1850 4800 2300 4800
 Text Label 4800 2150 0    50   ~ 0
 ISA_IRQ2
@@
 Wire Wire Line
 	6550 8950 6800 8950
-Wire Wire Line
-	1550 2400 1550 4500
 Connection ~ 1550 4500
 $Comp
 L Device:C C2
 U 1 1 61893822
-P 1000 6200
-F 0 "C2" H 1115 6246 50  0000 L CNN
-F 1 "47µF 10V" H 1115 6155 50  0000 L CNN
-F 2 "Capacitor_SMD:C_1206_3216Metric" H 1038 6050 50  0001 C CNN
-F 3 "~" H 1000 6200 50  0001 C CNN
-F 4 "C96123" H 1000 6200 50  0001 C CNN "LCSC"
-	1    1000 6200
+P 1000 4300
+F 0 "C2" H 1115 4346 50  0000 L CNN
+F 1 "47µF 10V" H 1115 4255 50  0000 L CNN
+F 2 "Capacitor_SMD:C_1206_3216Metric" H 1038 4150 50  0001 C CNN
+F 3 "~" H 1000 4300 50  0001 C CNN
+F 4 "C96123" H 1000 4300 50  0001 C CNN "LCSC"
+	1    1000 4300
 	1    0    0    -1
 $EndComp
@@
 L power:+5V #PWR0121
 U 1 1 618955B6
-P 1000 6000
-F 0 "#PWR0121" H 1000 5850 50  0001 C CNN
-F 1 "+5V" H 1015 6173 50  0000 C CNN
-F 2 "" H 1000 6000 50  0001 C CNN
-F 3 "" H 1000 6000 50  0001 C CNN
-	1    1000 6000
-	1    0    0    -1
-$EndComp
-Wire Wire Line
-	1000 6000 1000 6050
-Wire Wire Line
-	1000 6400 1550 6400
+P 1000 4100
+F 0 "#PWR0121" H 1000 3950 50  0001 C CNN
+F 1 "+5V" H 1015 4273 50  0000 C CNN
+F 2 "" H 1000 4100 50  0001 C CNN
+F 3 "" H 1000 4100 50  0001 C CNN
+	1    1000 4100
+	1    0    0    -1
+$EndComp
+Wire Wire Line
+	1000 4100 1000 4150
+Wire Wire Line
+	1000 4500 1550 4500
 Wire Wire Line
 	1550 1500 1550 2400
@@
 	7350 4400 7700 4400
 Wire Wire Line
-	1000 6350 1000 6400
+	1000 4450 1000 4500
 $Comp
 L Mechanical:MountingHole_Pad H4
@@
 	1    0    0    -1
 $EndComp
+$Comp
+L Connector:Bus_ISA_8bit J1
+U 1 1 6060D767
+P 3000 3000
+F 0 "J1" H 3000 4767 50  0000 C CNN
+F 1 "Bus_ISA_8bit" H 3000 4676 50  0000 C CNN
+F 2 "My_Components:Conn_Edge_PCB_ISA8" H 3000 3000 50  0001 C CNN
+F 3 "https://en.wikipedia.org/wiki/Industry_Standard_Architecture" H 3000 3000 50  0001 C CNN
+	1    3000 3000
+	1    0    0    -1
+$EndComp
+Wire Wire Line
+	1550 2400 1550 4500
+Wire Wire Line
+	1550 4700 1550 4500
+$Comp
+L power:GND #PWR0105
+U 1 1 5FB73D29
+P 1550 4700
+F 0 "#PWR0105" H 1550 4450 50  0001 C CNN
+F 1 "GND" H 1555 4527 50  0000 C CNN
+F 2 "" H 1550 4700 50  0001 C CNN
+F 3 "" H 1550 4700 50  0001 C CNN
+	1    1550 4700
+	1    0    0    -1
+$EndComp

Commit message: Redraw 8 bit board
Parts:
- removed C2: 47µF 10V, Capacitor_SMD:C_1206_3216Metric, symbol Device:C
- removed H1: MountingHole, ToolingHole:ToolingHole_JLCSMT, symbol Mechanical:MountingHole
- removed H5: OSHW Logo, Symbol:OSHW-Logo_11.4x12mm_Copper, symbol Mechanical:MountingHole
- removed Y1: 20MHz, Crystal:Crystal_SMD_3225-4Pin_3.2x2.5mm, symbol Device:Crystal_GND24
- added C2: 47uF, Capacitor_THT:CP_Radial_D5.0mm_P2.50mm, symbol Device:CP_Small
- added Y1: 20Mhz, Crystal:Crystal_HC49-4H_Vertical, symbol Device:Crystal_Small
- C1, C12, C15, C3, C4, C5, C6, C7: footprint Capacitor_SMD:C_0402_1005Metric -> Capacitor_THT:C_Disc_D6.0mm_W2.5mm_P5.00mm; LCSC C1525 -> (none)
- C10, C11, C13, C14: footprint Capacitor_SMD:C_1206_3216Metric -> Capacitor_THT:C_Disc_D6.0mm_W2.5mm_P5.00mm; LCSC C9196 -> (none)
- C8: footprint Capacitor_SMD:C_0402_1005Metric -> Capacitor_THT:C_Disc_D5.0mm_W2.5mm_P2.50mm; LCSC C1554 -> (none)
- C9: footprint Capacitor_SMD:C_0402_1005Metric -> Capacitor_THT:C_Disc_D5.0mm_W2.5mm_P2.50mm
- FB1: footprint Inductor_SMD:L_0805_2012Metric -> Inductor_THT:L_Axial_L5.3mm_D2.2mm_P10.16mm_Horizontal_Vishay_IM-1
- R1: footprint Resistor_SMD:R_0402_1005Metric -> Resistor_THT:R_Axial_DIN0207_L6.3mm_D2.5mm_P10.16mm_Horizontal; LCSC C25771 -> (none)
- R10, R11, R12, R13, R14, R15, R16, R17, R18, R19, R20, R21, R22, R6, R7, R8, R9: footprint Resistor_SMD:R_0402_1005Metric -> Resistor_THT:R_Axial_DIN0207_L6.3mm_D2.5mm_P10.16mm_Horizontal; LCSC C25744 -> (none)
- R2: footprint Resistor_SMD:R_0402_1005Metric -> Resistor_THT:R_Axial_DIN0207_L6.3mm_D2.5mm_P10.16mm_Horizontal; LCSC C26083 -> (none)
- R3: footprint Resistor_SMD:R_0402_1005Metric -> Resistor_THT:R_Axial_DIN0207_L6.3mm_D2.5mm_P10.16mm_Horizontal; LCSC C25087 -> (none)
- R4, R5: footprint Resistor_SMD:R_0402_1005Metric -> Resistor_THT:R_Axial_DIN0207_L6.3mm_D2.5mm_P10.16mm_Horizontal; LCSC C11702 -> (none)
Connections:
- net +5V: now also C2.1
- net GND: now also C2.2
- net at C8.2, R2.1, U1.50 (X1): now also Y1.2
- net at C9.2, R2.2, U1.51 (X2): now also Y1.1

Commit message: cleanup board a bit
Parts:
- C2: value 47uF -> 10uF
Changed lines of the file:
@@
 P 1000 4300
 F 0 "C2" H 1088 4346 50  0000 L CNN
-F 1 "47uF" H 1088 4255 50  0000 L CNN
+F 1 "10uF" H 1088 4255 50  0000 L CNN
 F 2 "Capacitor_THT:CP_Radial_D5.0mm_P2.50mm" H 1000 4300 50  0001 C CNN
 F 3 "~" H 1000 4300 50  0001 C CNN

Commit message: Add another filter cap
Parts:
- added C16: 10uF, Capacitor_THT:CP_Radial_D5.0mm_P2.50mm, symbol Device:CP_Small
Connections:
- net +5V: now also C16.1
- net GND: now also C16.2
Changed lines of the file:
@@
 $EndComp
 Wire Wire Line
-	1000 4100 1000 4200
+	1000 4100 1000 4150
 Wire Wire Line
 	1000 4400 1000 4500
+$Comp
+L Device:CP_Small C16
+U 1 1 607D3DB8
+P 650 4300
+F 0 "C16" H 738 4346 50  0000 L CNN
+F 1 "10uF" H 738 4255 50  0000 L CNN
+F 2 "Capacitor_THT:CP_Radial_D5.0mm_P2.50mm" H 650 4300 50  0001 C CNN
+F 3 "~" H 650 4300 50  0001 C CNN
+	1    650  4300
+	1    0    0    -1
+$EndComp
+Wire Wire Line
+	650  4200 650  4150
+Wire Wire Line
+	650  4150 1000 4150
+Connection ~ 1000 4150
+Wire Wire Line
+	1000 4150 1000 4200
+Wire Wire Line
+	650  4400 650  4500
+Wire Wire Line
+	650  4500 1000 4500
+Connection ~ 1000 4500
 $EndSCHEMATC

Commit message: Resize board and remove jumper for 16-bit IRQs
Parts:
- removed J9: IRQ select, Connector_PinHeader_2.54mm:PinHeader_2x03_P2.54mm_Vertical, symbol Connector_Generic:Conn_02x03_Odd_Even
- removed R22: 10k, Resistor_THT:R_Axial_DIN0207_L6.3mm_D2.5mm_P10.16mm_Horizontal, symbol Device:R
- added J9: IRQ select, Connector_PinHeader_2.54mm:PinHeader_2x02_P2.54mm_Vertical, symbol Connector_Generic:Conn_02x02_Odd_Even
- R1: value 27k -> 10k
Connections:
- net +5V: now also J9.2 (Pin_2), J9.4 (Pin_4)
- net at R21.2: now also J9.1 (Pin_1)
- net at R20.2: now also J9.3 (Pin_3)
Changed lines of the file:
@@
 P 4650 3400
 F 0 "R1" H 4580 3354 50  0000 R CNN
-F 1 "27k" H 4580 3445 50  0000 R CNN
+F 1 "10k" H 4580 3445 50  0000 R CNN
 F 2 "Resistor_THT:R_Axial_DIN0207_L6.3mm_D2.5mm_P10.16mm_Horizontal" V 4580 3400 50  0001 C CNN
 F 3 "~" H 4650 3400 50  0001 C CNN
@@
 $EndComp
 $Comp
-L Connector_Generic:Conn_02x03_Odd_Even J9
-U 1 1 605EED03
-P 14850 4400
-F 0 "J9" H 14900 4600 50  0000 C CNN
-F 1 "IRQ select" H 14900 4200 50  0000 C CNN
-F 2 "Connector_PinHeader_2.54mm:PinHeader_2x03_P2.54mm_Vertical" H 14850 4400 50  0001 C CNN
-F 3 "~" H 14850 4400 50  0001 C CNN
-	1    14850 4400
-	1    0    0    1
-$EndComp
-$Comp
 L Connector_Generic:Conn_02x01 J5
 U 1 1 60626BC2
@@
 	0    -1   -1   0
 $EndComp
-$Comp
-L Device:R R22
-U 1 1 608B4E30
-P 14350 4500
-F 0 "R22" H 14420 4546 50  0001 L CNN
-F 1 "10k" V 14350 4400 50  0000 L CNN
-F 2 "Resistor_THT:R_Axial_DIN0207_L6.3mm_D2.5mm_P10.16mm_Horizontal" V 14280 4500 50  0001 C CNN
-F 3 "~" H 14350 4500 50  0001 C CNN
-	1    14350 4500
-	0    -1   -1   0
-$EndComp
 Wire Wire Line
 	14500 1750 14650 1750
@@
 	14650 4400 14500 4400
 Wire Wire Line
-	14500 4500 14650 4500
-Wire Wire Line
 	15550 1750 15550 2100
 Wire Wire Line
@@
 Wire Wire Line
 	15550 1750 15150 1750
-Wire Wire Line
-	15550 4500 15150 4500
 Connection ~ 15550 2100
 Wire Wire Line
@@
 Wire Wire Line
 	15550 2100 15550 2450
-Connection ~ 15550 4400
-Wire Wire Line
-	15550 4400 15550 4500
 Wire Wire Line
 	15550 4300 15150 4300
@@
 Text Label 13950 4400 0    50   ~ 0
 IRQS1
-Text Label 13950 4500 0    50   ~ 0
-IRQS2
 Wire Wire Line
 	13950 4300 14200 4300
 Wire Wire Line
 	14200 4400 13950 4400
-Wire Wire Line
-	13950 4500 14200 4500
 Text Label 13950 3850 0    50   ~ 0
 PL0
@@
 	650  4500 1000 4500
 Connection ~ 1000 4500
+$Comp
+L Connector_Generic:Conn_02x02_Odd_Even J9
+U 1 1 60802B26
+P 14850 4400
+F 0 "J9" H 14900 4500 50  0000 C CNN
+F 1 "IRQ select" H 14900 4166 50  0000 C CNN
+F 2 "Connector_PinHeader_2.54mm:PinHeader_2x02_P2.54mm_Vertical" H 14850 4400 50  0001 C CNN
+F 3 "~" H 14850 4400 50  0001 C CNN
+	1    14850 4400
+	1    0    0    1
+$EndComp
 $EndSCHEMATC

Commit message: Removed useless pulldown resistor
Parts:
- removed R1: 10k, Resistor_THT:R_Axial_DIN0207_L6.3mm_D2.5mm_P10.16mm_Horizontal, symbol Device:R
Connections:
- net ~ISA_IOCS16 is gone; now on net GND: U1.96 (~IOCS16B~/SLOT16)
Changed lines of the file:
@@
 Wire Wire Line
 	4900 2000 5250 2000
-$Comp
-L Device:R R1
-U 1 1 5FB65FAE
-P 4650 3400
-F 0 "R1" H 4580 3354 50  0000 R CNN
-F 1 "10k" H 4580 3445 50  0000 R CNN
-F 2 "Resistor_THT:R_Axial_DIN0207_L6.3mm_D2.5mm_P10.16mm_Horizontal" V 4580 3400 50  0001 C CNN
-F 3 "~" H 4650 3400 50  0001 C CNN
-	1    4650 3400
-	1    0    0    1
-$EndComp
 Wire Wire Line
 	4650 3250 5250 3250
@@
 	1    0    0    1
 $EndComp
+Wire Wire Line
+	4650 3550 4650 3250
 $EndSCHEMATC

Commit message: Smaller version of the ethernet card
Parts:
- FB1: value Ferrite_Bead -> Filter
- R3: value 200R -> 200
- U3: footprint Package_DIP:DIP-32_W15.24mm_Socket_LongPads -> Package_DIP:DIP-32_W15.24mm_Socket
Changed lines of the file:
@@
 AR Path="/5FBE6809" Ref="R3"  Part="1"
 F 0 "R3" H 10970 8596 50  0000 L CNN
-F 1 "200R" H 10970 8505 50  0000 L CNN
+F 1 "200" H 10970 8505 50  0000 L CNN
 F 2 "Resistor_THT:R_Axial_DIN0207_L6.3mm_D2.5mm_P10.16mm_Horizontal" V 10830 8550 50  0001 C CNN
 F 3 "~" H 10900 8550 50  0001 C CNN
@@
 F 0 "U3" H 12350 3850 50  0000 C CNN
 F 1 "SST39SF010 / MX29F001T" V 12700 2550 50  0000 C CNN
-F 2 "Package_DIP:DIP-32_W15.24mm_Socket_LongPads" H 12700 2850 50  0001 C CNN
+F 2 "Package_DIP:DIP-32_W15.24mm_Socket" H 12700 2850 50  0001 C CNN
 F 3 "http://ww1.microchip.com/downloads/en/DeviceDoc/25022B.pdf" H 12700 2850 50  0001 C CNN
 	1    12700 2550
@@
 P 12550 9450
 F 0 "FB1" V 12276 9450 50  0000 C CNN
-F 1 "Ferrite_Bead" V 12367 9450 50  0000 C CNN
+F 1 "Filter" V 12367 9450 50  0000 C CNN
 F 2 "Inductor_THT:L_Axial_L5.3mm_D2.2mm_P10.16mm_Horizontal_Vishay_IM-1" V 12480 9450 50  0001 C CNN
 F 3 "~" H 12550 9450 50  0001 C CNN

Commit message: Added more IRQ options
Parts:
- removed J9: IRQ select, Connector_PinHeader_2.54mm:PinHeader_2x02_P2.54mm_Vertical, symbol Connector_Generic:Conn_02x02_Odd_Even
- added J9: IRQ Select, Connector_PinHeader_2.54mm:PinHeader_2x03_P2.54mm_Vertical, symbol Connector_Generic:Conn_02x03_Odd_Even
- added R22: 10k, Resistor_THT:R_Axial_DIN0207_L6.3mm_D2.5mm_P10.16mm_Horizontal, symbol Device:R
Connections:
- net ISA_IRQ10 is gone; now on net ISA_IRQ6: U1.100 (INT4)
- net ISA_IRQ11 is gone; now on net ISA_IRQ7: U1.99 (INT5)
- net +5V: now also J9.2 (Pin_2), J9.4 (Pin_4), J9.6 (Pin_6)
- net BD4: now also R22.1
- net at R21.2: now also J9.3 (Pin_3)
- net at R20.2: now also J9.5 (Pin_5)
- new net: J9.1 (Pin_1), R22.2
Changed lines of the file:
@@
 	4800 2250 5250 2250
 Text Label 4800 2550 0    50   ~ 0
-ISA_IRQ10
+ISA_IRQ6
 Text Label 4800 2650 0    50   ~ 0
-ISA_IRQ11
+ISA_IRQ7
 Text Label 4800 2750 0    50   ~ 0
 ISA_IRQ12
@@
 	14650 3950 14500 3950
 Wire Wire Line
-	14500 4300 14650 4300
-Wire Wire Line
-	14650 4400 14500 4400
-Wire Wire Line
 	15550 1750 15550 2100
 Wire Wire Line
@@
 Connection ~ 15550 2100
 Wire Wire Line
-	15150 4400 15550 4400
-Wire Wire Line
 	15550 2100 15550 2450
-Wire Wire Line
-	15550 4300 15150 4300
 Connection ~ 15550 4300
 Wire Wire Line
@@
 	650  4500 1000 4500
 Connection ~ 1000 4500
-$Comp
-L Connector_Generic:Conn_02x02_Odd_Even J9
-U 1 1 60802B26
+Wire Wire Line
+	4650 3550 4650 3250
+$Comp
+L Device:R R22
+U 1 1 60871D55
+P 14350 4500
+F 0 "R22" H 14420 4546 50  0001 L CNN
+F 1 "10k" V 14350 4400 50  0000 L CNN
+F 2 "Resistor_THT:R_Axial_DIN0207_L6.3mm_D2.5mm_P10.16mm_Horizontal" V 14280 4500 50  0001 C CNN
+F 3 "~" H 14350 4500 50  0001 C CNN
+	1    14350 4500
+	0    -1   -1   0
+$EndComp
+Wire Wire Line
+	14650 4500 14500 4500
+Text Label 13950 4500 0    50   ~ 0
+IRQS2
+Wire Wire Line
+	14200 4500 13950 4500
+Wire Wire Line
+	15550 4300 15150 4300
+Wire Wire Line
+	14500 4300 14650 4300
+Wire Wire Line
+	15150 4400 15550 4400
+Wire Wire Line
+	14650 4400 14500 4400
+$Comp
+L Connector_Generic:Conn_02x03_Odd_Even J9
+U 1 1 608CBD62
 P 14850 4400
-F 0 "J9" H 14900 4500 50  0000 C CNN
-F 1 "IRQ select" H 14900 4166 50  0000 C CNN
-F 2 "Connector_PinHeader_2.54mm:PinHeader_2x02_P2.54mm_Vertical" H 14850 4400 50  0001 C CNN
+F 0 "J9" H 14900 4600 50  0000 C CNN
+F 1 "IRQ Select" H 14900 4166 50  0000 C CNN
+F 2 "Connector_PinHeader_2.54mm:PinHeader_2x03_P2.54mm_Vertical" H 14850 4400 50  0001 C CNN
 F 3 "~" H 14850 4400 50  0001 C CNN
 	1    14850 4400
@@
 $EndComp
 Wire Wire Line
-	4650 3550 4650 3250
+	15150 4500 15550 4500
+Wire Wire Line
+	15550 4500 15550 4400
+Connection ~ 15550 4400
 $EndSCHEMATC
